Commit message: Update igvc_bot.urdf

File: urdf/igvc_bot.urdf (robot description, URDF)
Before this commit: robot bot2, 7 links, 6 joints
Links:
- link base_link: mass 8 -> 6

Commit message: two default camera. Should it be stereo?

File: urdf/igvc_bot.urdf (robot description, URDF)
Before this commit: robot bot, 7 links, 6 joints
Links:
- added link camera_left; visual box size=0.05 0.05 0.05
- added link camera_right; visual box size=0.05 0.05 0.05
Joints:
- added joint camera_left: type fixed, parent base_link, child camera_left, origin xyz=0.72 -0.05 1.175 rpy=0 0 0, limit effort=2 velocity=5
- added joint camera_right: type fixed, parent base_link, child camera_right, origin xyz=0.72 0.05 1.175 rpy=0 0 0, limit effort=2 velocity=5

Commit message: imu

File: urdf/igvc_bot.urdf (robot description, URDF)
Before this commit: robot bot, 9 links, 8 joints
Links:
- added link imu_link; visual box size=0.02 0.02 0.02
Joints:
- added joint imu: type fixed, parent base_link, child imu_link, origin xyz=0 0 0.39 rpy=0 0 0, limit effort=2 velocity=5

Commit message: gps

File: urdf/igvc_bot.urdf (robot description, URDF)
Before this commit: robot bot, 10 links, 9 joints
Links:
- added link gps_link
Joints:
- added joint gps_joint: type fixed, parent base_link, child gps_link, origin xyz=0 0 0

Commit message: Switched to two camera detection

File: urdf/igvc_bot.urdf (robot description, URDF)
Before this commit: robot bot, 11 links, 10 joints
Joints:
- joint camera_left: origin xyz=0.72 -0.05 1.175 rpy=0 0 0 -> xyz=0.72 -0.05 1.175 rpy=0 0 -0.5
- joint camera_right: origin xyz=0.72 0.05 1.175 rpy=0 0 0 -> xyz=0.72 0.05 1.175 rpy=0 0 0.5

Commit message: minor edit

File: urdf/igvc_bot.urdf (robot description, URDF)
Before this commit: robot bot, 11 links, 10 joints
Joints:
- joint camera_left: origin xyz=0.72 -0.05 1.175 rpy=0 0 -0.5 -> xyz=0.72 -0.05 1.175 rpy=0 0 -0.6
- joint camera_right: origin xyz=0.72 0.05 1.175 rpy=0 0 0.5 -> xyz=0.72 0.05 1.175 rpy=0 0 0.6

Commit message: small changes

File: urdf/igvc_bot.urdf (robot description, URDF)
Before this commit: robot bot, 11 links, 10 joints
Joints:
- joint camera_left: origin xyz=0.72 -0.05 1.175 rpy=0 0 -0.6 -> xyz=0.72 0.05 1.175 rpy=0 0 0.6
- joint camera_right: origin xyz=0.72 0.05 1.175 rpy=0 0 0.6 -> xyz=0.72 -0.05 1.175 rpy=0 0 -0.6

Commit message: tried a lane continuation system big problems

File: urdf/igvc_bot.urdf (robot description, URDF)
Before this commit: robot bot, 11 links, 10 joints
Joints:
- joint camera_left: origin xyz=0.72 0.05 1.175 rpy=0 0 0.6 -> xyz=0.72 0.05 1.175 rpy=0 0.1 0.6
- joint camera_right: origin xyz=0.72 -0.05 1.175 rpy=0 0 -0.6 -> xyz=0.72 -0.05 1.175 rpy=0 0.1 -0.6
